File: IgnitionBoardV1/IgnitionBoardV1.kicad_pcb (KiCad board)
At the start: 2 copper layers, 45 x 45 mm, 12 parts, among them J1 Screw_Terminal_01x02, J2 Screw_Terminal_01x02, J3 Screw_Terminal_01x02, J4 Screw_Terminal_01x02, J5 Screw_Terminal_01x02, Q1 NMOS, Q2 NMOS

Commit message: Add board name and version to silkscreen
Parts:
- moved LOGO_SOAR 5.51 mm to (157.8, 62.0)
Other:
- board text added: "Ignition / Trigger Board V1"
Changed lines of the file:
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@@
 (kicad_pcb (version 4) (host pcbnew 4.0.7)
   (general
-    (links 16)
+    (links 0)
     (no_connects 0)
-    (area 113 21 181.000001 87.000001)
+    (area 124.924999 29.924999 170.075001 75.075001)
     (thickness 1.6)
-    (drawings 82)
+    (drawings 83)
     (tracks 16)
     (zones 0)
@@
   (layers
     (0 F.Cu signal)
-    (31 B.Cu signal)
+    (31 B.Cu signal hide)
     (32 B.Adhes user)
     (33 F.Adhes user)
@@
   )
   (module SOAR_LOGO_KICAD:LOGO_SOAR (layer F.Cu)
-    (at 158 67.5)
-    (fp_text reference LOGO_SOAR (at 8 8.5) (layer F.SilkS) hide
+    (at 157.75 62)
+    (fp_text reference LOGO_SOAR (at 5.75 -1) (layer F.SilkS) hide
       (effects (font (thickness 0.3)))
     )
@@
       (xy 5.75 5.1)) (layer F.SilkS) (width 0.01))
   )
+  (gr_text "Ignition / \nTrigger Board\nV1" (at 159 70.75) (layer F.SilkS)
+    (effects (font (size 1 1) (thickness 0.2)) (justify left))
+  )
   (gr_line (start 163 40.3) (end 159.1 40.3) (layer B.SilkS) (width 0.2))

Commit message: Generated gerbers
Parts:
- moved LOGO_SOAR 0.53 mm to (157.4, 62.4)
- moved J2 0.10 mm to (130.0, 69.4)
Other:
- board text added: "Ignition & Trigger Board V1 (May 2018)"
- board text removed: "Ignition / Trigger Board V1"
Changed lines of the file:
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@@
 (kicad_pcb (version 4) (host pcbnew 4.0.7)
   (general
-    (links 0)
+    (links 16)
     (no_connects 0)
-    (area 124.924999 29.924999 170.075001 75.075001)
+    (area 113 21 181.000001 87.000001)
     (thickness 1.6)
     (drawings 83)
@@
   (layers
     (0 F.Cu signal)
-    (31 B.Cu signal hide)
+    (31 B.Cu signal)
     (32 B.Adhes user)
     (33 F.Adhes user)
@@
     (last_trace_width 0.4)
     (trace_clearance 0.2)
-    (zone_clearance 0.508)
+    (zone_clearance 0.4)
     (zone_45_only yes)
     (trace_min 0.2)
@@
     (pcbplotparams
       (layerselection 0x000f0_80000001)
-      (usegerberextensions true)
+      (usegerberextensions false)
       (excludeedgelayer false)
       (linewidth 0.100000)
@@
   )
   (module TerminalBlock_Phoenix:TerminalBlock_Phoenix_PT-1,5-2-5.0-H_1x02_P5.00mm_Horizontal (layer F.Cu)
-    (at 130 69.5)
+    (at 130 69.4)
     (descr "Terminal Block Phoenix PT-1,5-2-5.0-H, 2 pins, pitch 5.0mm, size 10.0x9mm^2, drill diamater 1.3mm, pad diameter 2.6mm, see http://www.mouser.com/ds/2/324/ItemDetail_1935161-922578.pdf, script-generated using https://github.com/pointhi/kicad-footprint-generator/scripts/TerminalBlock_Phoenix")
     (tags "THT Terminal Block Phoenix PT-1.5-2-5.0-H pitch 5.0mm size 10.0x9mm^2 drill 1.3mm pad 2.6mm")
@@
   )
   (module SOAR_LOGO_KICAD:LOGO_SOAR (layer F.Cu)
-    (at 157.75 62)
+    (at 157.4 62.4)
     (fp_text reference LOGO_SOAR (at 5.75 -1) (layer F.SilkS) hide
       (effects (font (thickness 0.3)))
@@
       (xy 5.75 5.1)) (layer F.SilkS) (width 0.01))
   )
-  (gr_text "Ignition / \nTrigger Board\nV1" (at 159 70.75) (layer F.SilkS)
+  (gr_text "Ignition &\nTrigger Board\nV1 (May 2018)" (at 158.6 70.4) (layer F.SilkS)
     (effects (font (size 1 1) (thickness 0.2)) (justify left))
   )
@@
   (segment (start 155.76 54.46) (end 151.5 54.46) (width 0.4) (layer B.Cu) (net 8))
   (zone (net 4) (net_name VDD) (layer F.Cu) (hatch edge 0.508)
-    (connect_pads yes (clearance 0.25))
+    (connect_pads yes (clearance 0.4))
     (min_thickness 0.5)
     (fill yes (arc_segments 16) (thermal_gap 0.508) (thermal_bridge_width 1))
@@
   (zone (net 6) (net_name "Net-(J4-Pad1)") (layer F.Cu) (hatch edge 0.508)
     (priority 1)
-    (connect_pads yes (clearance 0.25))
+    (connect_pads yes (clearance 0.3))
     (min_thickness 0.3)
     (fill yes (arc_segments 16) (thermal_gap 0.5) (thermal_bridge_width 1))
@@
   (zone (net 3) (net_name "Net-(J2-Pad1)") (layer F.Cu) (hatch edge 0.508)
     (priority 1)
-    (connect_pads yes (clearance 0.25))
+    (connect_pads yes (clearance 0.3))
     (min_thickness 0.3)
     (fill yes (arc_segments 16) (thermal_gap 0.5) (thermal_bridge_width 1))
     (polygon
       (pts
-        (xy 137.5 50.5) (xy 124.75 50.5) (xy 124 75.5) (xy 133 75) (xy 133 65)
-        (xy 133 58.5) (xy 137.25 58.5)
-      )
-    )
-  )
-  (zone (net 3) (net_name "Net-(J2-Pad1)") (layer F.Cu) (hatch edge 0.508)
-    (priority 1)
-    (connect_pads yes (clearance 0.25))
-    (min_thickness 0.3)
-    (fill yes (arc_segments 16) (thermal_gap 0.5) (thermal_bridge_width 1))
-    (polygon
-      (pts
-        (xy 127 66.5) (xy 132.5 66.5) (xy 132.5 74.5) (xy 127 74.5)
+        (xy 137.25 58.5) (xy 133 58.5) (xy 133 75) (xy 124 75.5) (xy 124.75 50.5)
+        (xy 137.5 50.5)
       )
     )
